File: PCB_2.kicad_sch (KiCad schematic)
At the start: 19 parts, among them Q3 Q_NPN_BCE, Q4 Q_NPN_BCE, U3 TEA1-0505

Commit message: Updated schematic and layout, cleaned backups
Parts:
- removed Q3, Q4: Q_NPN_BCE, Package_TO_SOT_THT:TO-92_Inline, symbol Transistor_BJT:Q_NPN_BCE
- added C6: 10u, Capacitor_SMD:C_0805_2012Metric, symbol Device:C_Small
- added D3: D_Photo, Diode_SMD:D_0805_2012Metric_Pad1.15x1.40mm_HandSolder, symbol Device:D_Photo
- added Q1, Q2: BC817, Package_TO_SOT_SMD:SOT-23, symbol Transistor_BJT:BC817
- C3: value 10 nF -> 10n
- C4: value C_Small -> 10u
- C5: value 10 uF -> 10u
- P1: renamed from Potentiometer3; footprint Potentiometer_THT:Potentiometer_ACP_CA9-V10_Vertical_Hole -> Potentiometer_SMD:Potentiometer_Bourns_3214W_Vertical
- P2: renamed from Potentiometer4; footprint Potentiometer_THT:Potentiometer_ACP_CA9-V10_Vertical_Hole -> Potentiometer_SMD:Potentiometer_Bourns_3214W_Vertical
- R25: value 1 MΩ -> 1M
- R26: value 1000 Ω -> 1k
- renumbered Digital_Out1 to Input, Analog_In1 to Output
Connections:
- net +5V: now also D3.2 (A)
- net -5V: now also C6.2
- net GND: now also Input.5 (Pin_5), OPA828.3 (+), C6.1, Q1.2 (E), Q2.2 (E)
- net at LED_ir_(950nm)_SMD1.1 (K), LED_ir_(950nm)_THT1.1 (K): now also Q2.3 (C)
- net at P2.2: now also Q2.1 (B)
- net at OPA828.2 (-), R25.1: now also D2.1 (K), D3.1 (K)
- net at P1.2: now also Q1.1 (B)
- net at LED_red_(640nm)_SMD1.1 (K), LED_red_(640nm)_THT1.1 (K): now also Q1.3 (C)
Other:
- moved on the sheet: C4, D2, R25, U3
